File: twoboPICard/PI_Card v2.kicad_pcb (KiCad board)
At the start: 4 copper layers, 110 x 75 mm, 22 parts, among them J1 Conn_02x20_Odd_Even, J2 Conn_02x20_Odd_Even, J3 Conn_01x03_Pin, J4 Conn_01x02, J5 Conn_02x40_Odd_Even, J6 Conn_01x03_Pin, SW1 SW_Push

Commit message: Fixed Fuse Positioning & Unconnected Nets
Parts:
- moved F1 69.0 mm to (243.1, 51.7), turned to 180 degrees
- moved D4 27.3 mm to (197.7, 49.9)
- moved G*** 15.0 mm to (200.6, 77.2)
- moved G*** 3.95 mm to (200.2, 79.8)
- moved C1 2.43 mm to (255.3, 58.7)
- moved D2 1.93 mm to (256.2, 69.3)
- moved D3 1.75 mm to (256.3, 78.7)
- moved R2 1.68 mm to (249.6, 69.2)
- moved D1 1.44 mm to (256.4, 87.9)
- moved R3 1.36 mm to (249.7, 78.6)
- moved R1 1.05 mm to (249.4, 87.9)
Routing:
- net +3V3: track 0.00 -> 52.4 mm, vias 0 -> 4
- net GPIO17: track 76.8 -> 103.7 mm
- net GND: track 0.00 -> 19.2 mm
- net Net-(D3-A): track 4.31 -> 3.13 mm
- net Net-(D2-A): track 4.03 -> 3.14 mm
- net Net-(D1-A): track 4.22 -> 3.58 mm
- net +5V: vias 12 -> 11
Other:
- board text added: "+3V3"
- board text added: "+5V"
- board text added: "ALIVE"
