File: quboPowerCard/_autosave-quboPowerCard.kicad_sch (KiCad schematic)
At the start: 17 parts, among them J2 Conn_01x09, J5 Conn_02x40_Odd_Even

Commit message: Repositioned Mounting Holes
Parts:
- removed A1, A2, A3: SolderJumper_2_Open, Jumper:SolderJumper-2_P1.3mm_Open_TrianglePad1.0x1.5mm, symbol Jumper:SolderJumper_2_Open
- removed C2: 10u, Capacitor_SMD:C_0805_2012Metric_Pad1.18x1.45mm_HandSolder, symbol Device:C
- removed D1: LED_RGAB, LED_THT:LED_D5.0mm-4_RGB, symbol Device:LED_RGAB
- removed H1, H2, H3: MountingHole, MountingHole:MountingHole_2.2mm_M2, symbol Mechanical:MountingHole
- removed I2C_PWM_DRIVER1: PCA9685, Package_SO:TSSOP-28_4.4x9.7mm_P0.65mm, symbol New_Library:PCA9685
- removed J2: Conn_01x09, Connector_Molex:Molex_Micro-Fit_3.0_43650-0900_1x09_P3.00mm_Horizontal, symbol Connector_Generic:Conn_01x09
- removed R1, R2, R3: 220, Resistor_SMD:R_0805_2012Metric_Pad1.20x1.40mm_HandSolder, symbol Device:R
- removed U2, U3, U4: ~, custom_components:ESC_blue_robotics, symbol Thruster_Control_Components:ESC
- added C1, C3, C6: 1u, Capacitor_SMD:C_0805_2012Metric_Pad1.18x1.45mm_HandSolder, symbol PowerboardRev5-eagle-import:C-USC0805
- added J1, J2: Conn_01x02_Pin, customRAM:JST_PH_B2B-PH-K_1x02_P2.00mm_Vertical, symbol Connector:Conn_01x02_Pin
- added J4: Conn_01x04_Pin, customRAM:1.25__FUSECLIPS, symbol Connector:Conn_01x04_Pin
- added J6: 1720420202, customRAM:SUPERSABRE_2CIRCUIT, symbol supersabre:1720420202
- added PS1: THL_25-2411WI, customRAM:CONV_THL_25-2411WI, symbol customRAM:THL_25-2411WI
- added Q1, Q2: IRF5305PbF, Package_TO_SOT_THT:TO-220-3_Vertical, symbol Transistor_FET:FQP27P06
- added R1, R6: 10kO, Resistor_SMD:R_0805_2012Metric_Pad1.20x1.40mm_HandSolder, symbol PowerboardRev5-eagle-import:R-US_R0805
- added U1: ~, customRAM:240W_CONV, symbol Custom:PKB2213D
- added U3: TSR2-2450, customRAM:CONV_TSR_2-2450, symbol PowerboardRev5-eagle-import:TSR2-2450
- added U4: TSR2-2433, customRAM:CONV_TSR2-2433, symbol PowerboardRev5-eagle-import:TSR2-2450
- J5: footprint Samtec Custom:Samtec_HLE-140-02-L-DV-PE_2x40_P2.54mm_Horizontal -> Connector_PinHeader_1.00mm:PinHeader_2x40_P1.00mm_Vertical
Connections:
- net +12V: now also U1.8 (VOUT)
- net +3.3V: now also C6.1, U4.3 (+V_OUT)
- net +5V: now also C3.1, U3.3 (+V_OUT)
- net GND: now also C1.2, C3.2, C6.2, J1.2 (Pin_2), J2.2 (Pin_2), J6.2, PS1.2 (-VIN(GND)), U1.3 (IN-), U1.4 (OUT-), U3.2 (GND), U4.2 (GND)
- net PiPower5V: now reaches J5.41 (Pin_41)
- net PiPower5V: now also J5.42 (Pin_42), J5.43 (Pin_43), J5.44 (Pin_44), J5.45 (Pin_45), J5.46 (Pin_46), C1.1, PS1.3 (+VOUT)
- net SCL: no longer names the net of J5.1 (Pin_1)
- net SDA: no longer names the net of J5.3 (Pin_3)
- new net: J4.1 (Pin_1), J4.2 (Pin_2), Q1.2 (D)
- new net +24V: J6.1, Q1.3 (S), R1.1
- new net NPSW1: J1.1 (Pin_1), Q2.1 (G), R6.2
- new net NonPiPower: Q2.2 (D), U1.1 (VIN), U3.1 (+V_IN), U4.1 (+V_IN)
- new net SW2: J2.1 (Pin_1), Q1.1 (G), R1.2
- new net V_POWER: J4.3 (Pin_3), J4.4 (Pin_4), PS1.1 (+VIN(VCC)), Q2.3 (S), R6.1
- no-connect marks 62 -> 0
Other:
- note added: "24V Connector"
- note added: "Convert to 3.3V"
- note added: "Convert to 5V"
- note added: "Convert to 5V for Pi"
- note added: "Everything But Pi Kill Switch"
- note added: "Kill Switch and fuse"
- note removed: "ESC"
- note removed: "Stackup Connector"
- moved on the sheet: J5
