File: twoboThrusterCard/twobo_thrusters/twobo_thrusters.kicad_pcb (KiCad board)
At the start: 4 copper layers, 110 x 75 mm, 14 parts, among them J2 Conn_01x09, J5 Conn_02x40_Odd_Even

Commit message: twoBo thruster
Routing:
- net Net-(A3-B): track 0.00 -> 18.9 mm
- net Net-(A2-B): track 0.00 -> 14.8 mm
- net Net-(A1-B): track 0.00 -> 9.12 mm
- net GND: track 1.95 -> 3.82 mm, vias 67 -> 141
- added copper zone on F.Cu, net GND
- removed copper zone on F.Cu, net /A3
