File: PI Card/PI_Card v2.kicad_pcb (KiCad board)
At the start: 4 copper layers, 110 x 75 mm, 29 parts, among them J1 Conn_02x20_Odd_Even, J10 Conn_01x02_Pin, J11 Conn_01x02, J12 Conn_01x02_Pin, J2 Conn_02x20_Odd_Even, J3 Conn_01x03_Pin, J4 Conn_01x02, J5 Conn_02x40_Odd_Even, J6 Conn_01x03_Pin, J7 Conn_01x02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

Commit message: Added I2C Pull Up Resistors
Parts:
- added R4: 4.7k, Resistor_SMD:R_0805_2012Metric_Pad1.20x1.40mm_HandSolder, F.Cu at (236.6, 69.3)
- added R5: 4.7k, Resistor_SMD:R_0805_2012Metric_Pad1.20x1.40mm_HandSolder, F.Cu at (236.5, 65.7)
Routing:
- net SCL: track 54.6 -> 82.4 mm
- net SDA: track 35.5 -> 50.4 mm
- net +3V3: track 69.9 -> 81.6 mm
